Commit message: trying to implement ppo

File: urdf/ruff.urdf (robot description, URDF)
Before this commit: robot ruff, 14 links, 13 joints
Links:
- removed link imu_link
Joints:
- removed joint IMU_joint

Commit message: fixed limit bug in urdf file

File: urdf/ruff.urdf (robot description, URDF)
Before this commit: robot ruff, 13 links, 12 joints
Joints:
- joint FL1_: limit lower=0 upper=3.14 effort=200 velocity=10 -> lower=-0.785398 upper=0.785398 effort=200 velocity=10
- joint FL2_: limit lower=0 upper=3.14 effort=200 velocity=10 -> lower=-0.785398 upper=0.785398 effort=200 velocity=10
- joint FL3_: limit lower=0 upper=3.14 effort=200 velocity=10 -> lower=-0.785398 upper=0.785398 effort=200 velocity=10
- joint FR1_: limit lower=0 upper=3.14 effort=200 velocity=10 -> lower=-0.785398 upper=0.785398 effort=200 velocity=10
- joint FR2_: limit lower=0 upper=3.14 effort=200 velocity=10 -> lower=-0.785398 upper=0.785398 effort=200 velocity=10
- joint FR3_: limit lower=0 upper=3.14 effort=200 velocity=10 -> lower=-0.785398 upper=0.785398 effort=200 velocity=10
- joint RL1_: limit lower=0 upper=3.14 effort=200 velocity=10 -> lower=-0.785398 upper=0.785398 effort=200 velocity=10
- joint RL2_: limit lower=0 upper=3.14 effort=200 velocity=10 -> lower=-0.785398 upper=0.785398 effort=200 velocity=10
- joint RL3_: limit lower=0 upper=3.14 effort=200 velocity=10 -> lower=-0.785398 upper=0.785398 effort=200 velocity=10
- joint RR1_: limit lower=0 upper=3.14 effort=200 velocity=10 -> lower=-0.785398 upper=0.785398 effort=200 velocity=10
- joint RR2_: limit lower=0 upper=3.14 effort=200 velocity=10 -> lower=-0.785398 upper=0.785398 effort=200 velocity=10
- joint RR3_: limit lower=0 upper=3.14 effort=200 velocity=10 -> lower=-0.785398 upper=0.785398 effort=200 velocity=10

Commit message: fixed bug in actor loss

File: urdf/ruff.urdf (robot description, URDF)
Before this commit: robot ruff, 13 links, 12 joints
Joints:
- joint FL1_: limit lower=-0.785398 upper=0.785398 effort=200 velocity=10 -> lower=0 upper=0 effort=200 velocity=10
- joint FR1_: limit lower=-0.785398 upper=0.785398 effort=200 velocity=10 -> lower=0 upper=0 effort=200 velocity=10
- joint RL1_: limit lower=-0.785398 upper=0.785398 effort=200 velocity=10 -> lower=0 upper=0 effort=200 velocity=10
- joint RR1_: limit lower=-0.785398 upper=0.785398 effort=200 velocity=10 -> lower=0 upper=0 effort=200 velocity=10

Commit message: works but faulty buffer

File: urdf/ruff.urdf (robot description, URDF)
Before this commit: robot ruff, 13 links, 12 joints
Joints:
- joint FL1_: limit lower=0 upper=0 effort=200 velocity=10 -> lower=-0.174532 upper=0.174532 effort=200 velocity=10
- joint FL2_: limit lower=-0.785398 upper=0.785398 effort=200 velocity=10 -> lower=-0.174532 upper=0.174532 effort=200 velocity=10
- joint FL3_: limit lower=-0.785398 upper=0.785398 effort=200 velocity=10 -> lower=-0.52359 upper=0.52359 effort=200 velocity=10
- joint FR1_: limit lower=0 upper=0 effort=200 velocity=10 -> lower=-0.174532 upper=0.174532 effort=200 velocity=10
- joint FR2_: limit lower=-0.785398 upper=0.785398 effort=200 velocity=10 -> lower=-0.174532 upper=0.174532 effort=200 velocity=10
- joint FR3_: limit lower=-0.785398 upper=0.785398 effort=200 velocity=10 -> lower=-0.52359 upper=0.52359 effort=200 velocity=10
- joint RL1_: limit lower=0 upper=0 effort=200 velocity=10 -> lower=-0.174532 upper=0.174532 effort=200 velocity=10
- joint RL2_: limit lower=-0.785398 upper=0.785398 effort=200 velocity=10 -> lower=-0.174532 upper=0.174532 effort=200 velocity=10
- joint RL3_: limit lower=-0.785398 upper=0.785398 effort=200 velocity=10 -> lower=-0.52359 upper=0.52359 effort=200 velocity=10
- joint RR1_: limit lower=0 upper=0 effort=200 velocity=10 -> lower=-0.174532 upper=0.174532 effort=200 velocity=10
- joint RR2_: limit lower=-0.785398 upper=0.785398 effort=200 velocity=10 -> lower=-0.174532 upper=0.174532 effort=200 velocity=10
- joint RR3_: limit lower=-0.785398 upper=0.785398 effort=200 velocity=10 -> lower=-0.52359 upper=0.52359 effort=200 velocity=10

Commit message: works

File: urdf/ruff.urdf (robot description, URDF)
Before this commit: robot ruff, 13 links, 12 joints
Joints:
- joint FL1_: limit lower=-0.174532 upper=0.174532 effort=200 velocity=10 -> lower=0 upper=0 effort=200 velocity=10
- joint FR1_: limit lower=-0.174532 upper=0.174532 effort=200 velocity=10 -> lower=0 upper=0 effort=200 velocity=10
- joint RL1_: limit lower=-0.174532 upper=0.174532 effort=200 velocity=10 -> lower=0 upper=0 effort=200 velocity=10
- joint RR1_: limit lower=-0.174532 upper=0.174532 effort=200 velocity=10 -> lower=0 upper=0 effort=200 velocity=10

Commit message: manual restraint

File: urdf/ruff.urdf (robot description, URDF)
Before this commit: robot ruff, 13 links, 12 joints
Joints:
- joint FL2_: limit lower=-0.174532 upper=0.174532 effort=200 velocity=10 -> lower=-0.52333 upper=0.52333 effort=200 velocity=10
- joint FL3_: limit lower=-0.52359 upper=0.52359 effort=200 velocity=10 -> lower=-0.52333 upper=0.52333 effort=200 velocity=10
- joint FR2_: limit lower=-0.174532 upper=0.174532 effort=200 velocity=10 -> lower=-0.52333 upper=0.52333 effort=200 velocity=10
- joint FR3_: limit lower=-0.52359 upper=0.52359 effort=200 velocity=10 -> lower=-0.52333 upper=0.52333 effort=200 velocity=10
- joint RL2_: limit lower=-0.174532 upper=0.174532 effort=200 velocity=10 -> lower=-0.52333 upper=0.52333 effort=200 velocity=10
- joint RL3_: limit lower=-0.52359 upper=0.52359 effort=200 velocity=10 -> lower=-0.52333 upper=0.52333 effort=200 velocity=10
- joint RR2_: limit lower=-0.174532 upper=0.174532 effort=200 velocity=10 -> lower=-0.52333 upper=0.52333 effort=200 velocity=10
- joint RR3_: limit lower=-0.52359 upper=0.52359 effort=200 velocity=10 -> lower=-0.52333 upper=0.52333 effort=200 velocity=10

Commit message: minor changes

File: urdf/ruff.urdf (robot description, URDF)
Before this commit: robot ruff, 13 links, 12 joints
Links:
- link FL1: geometry collision mesh filename=../meshes/FL1.STL; visual mesh filename=../meshes/FL1.STL
- link FL2: geometry collision mesh filename=../meshes/FL2.STL; visual mesh filename=../meshes/FL2.STL
- link FL3: geometry collision mesh filename=../meshes/FL3.STL; visual mesh filename=../meshes/FL3.STL
- link FR1: geometry collision mesh filename=../meshes/FR1.STL; visual mesh filename=../meshes/FR1.STL
- link FR2: geometry collision mesh filename=../meshes/FR2.STL; visual mesh filename=../meshes/FR2.STL
- link FR3: geometry collision mesh filename=../meshes/FR3.STL; visual mesh filename=../meshes/FR3.STL
- link RL1: geometry collision mesh filename=../meshes/RL1.STL; visual mesh filename=../meshes/RL1.STL
- link RL2: geometry collision mesh filename=../meshes/RL2.STL; visual mesh filename=../meshes/RL2.STL
- link RL3: geometry collision mesh filename=../meshes/RL3.STL; visual mesh filename=../meshes/RL3.STL
- link RR1: geometry collision mesh filename=../meshes/RR1.STL; visual mesh filename=../meshes/RR1.STL
- link RR2: geometry collision mesh filename=../meshes/RR2.STL; visual mesh filename=../meshes/RR2.STL
- link RR3: geometry collision mesh filename=../meshes/RR3.STL; visual mesh filename=../meshes/RR3.STL
- link base_link: geometry collision mesh filename=../meshes/base_link.STL; visual mesh filename=../meshes/base_link.STL

Commit message: it runssgit add *

File: urdf/ruff.urdf (robot description, URDF)
Before this commit: robot ruff, 13 links, 12 joints
Joints:
- joint FL1_: limit lower=0 upper=0 effort=200 velocity=10 -> lower=-0.785 upper=0.785 effort=200 velocity=10
- joint FR1_: limit lower=0 upper=0 effort=200 velocity=10 -> lower=-0.785 upper=0.785 effort=200 velocity=10
- joint RL1_: limit lower=0 upper=0 effort=200 velocity=10 -> lower=-0.785 upper=0.785 effort=200 velocity=10
- joint RR1_: limit lower=0 upper=0 effort=200 velocity=10 -> lower=-0.785 upper=0.785 effort=200 velocity=10
