Commit message: switched to new ruff model

File: urdf/ruff_new.urdf (robot description, URDF)
Before this commit: robot bones, 18 links, 17 joints
Joints:
- joint FL1_: type continuous -> revolute
- joint FL2_: type continuous -> revolute
- joint FL3_: type continuous -> revolute
- joint FR1_: type continuous -> revolute
- joint FR2_: type continuous -> revolute
- joint FR3_: type continuous -> revolute
- joint RL1_: type continuous -> revolute
- joint RL2_: type continuous -> revolute
- joint RL3_: type continuous -> revolute
- joint RR1_: type continuous -> revolute
- joint RR2_: type continuous -> revolute
- joint RR3_: type continuous -> revolute

Commit message: fixxed bugs with updated urdf

File: urdf/ruff_new.urdf (robot description, URDF)
Before this commit: robot bones, 18 links, 17 joints
Links:
- removed link root_link
Joints:
- removed joint root_joint
